File: TXRX_relay_board.kicad_pcb (KiCad board)
At the start: 2 copper layers, 100 x 82 mm, 80 parts, among them J1 Screw_Terminal_01x02, J2 Conn_01x08, J3 IN, J4 IN_RF_Deck, J5 OUT_RF_Deck, J6 OUT, K1 RT314A05, K2 RT314A05, Q1 MMSS8550HE3, Q2 MMSS8550HE3, Q3 BC847, Q4 PNP, Q5 MMSS8550HE3, Q6 PNP, U1 OP07, U2 AMS1117-5.0

Commit message: rev 1.2
Minor fixes, coupler measurements, falstad simulation of over power protection
Parts:
- removed the REF** at (87.6, 76.3) (x2)
- added REF**: OSHW-Logo2_14.6x12mm_SilkScreen, Symbol:OSHW-Logo2_14.6x12mm_SilkScreen, F.Cu at (88.9, 74.0)
- added REF**: OSHW-Logo2_14.6x12mm_SilkScreen, Symbol:OSHW-Logo2_14.6x12mm_SilkScreen, B.Cu at (88.9, 74.0)
- Q1, Q2, Q5: value MMSS8550HE3 -> BC807
- Q3: value BC847 -> BC846
- Q4, Q6: value PNP -> BC807
- moved U1 0.29 mm to (89.9, 122.3)
- moved Q2 0.20 mm to (130.2, 62.3)
- moved Q3 0.20 mm to (93.9, 128.6)
- moved U2 0.19 mm to (73.9, 96.2)
- moved Q4 0.18 mm to (102.6, 132.7)
- moved Q5 0.11 mm to (102.8, 128.7)
- moved Q6 0.10 mm to (102.7, 136.3)
- renumbered C11 to C10, C12 to C11, C13 to C12, C14 to C13, C15 to C14, C16 to C15, C17 to C16, C18 to C17, C19 to C18, C20 to C19, C3 to C2, C21 to C20, C22 to C21, C23 to C22, C24 to C23, C4 to C3, C5 to C4, C6 to C5, C7 to C6, C8 to C7, C9 to C8, C10 to C9
Routing:
- net FWD_PWR: track 53.9 -> 45.9 mm, vias 1 -> 0
- net Net-(C3-Pad1): track 11.2 -> 8.63 mm
- net Net-(K1-Pad12): track 35.5 -> 37.2 mm
- net Net-(J5-In): track 18.8 -> 18.0 mm
- net +5V: track 58.0 -> 58.5 mm
- net GND: vias 406 -> 442
Other:
- board text added: "0,0000 mm / 0,0000 mm"
- board text added: "0,3000 mm"
- board text added: "1,6000 mm"
- board text added: "100,0000 mm x 82,0000 mm"
- board text added: "2"
- board text added: "BOARD CHARACTERISTICS"
- board text added: "Board Thickness:"
- board text added: "Board overall dimensions:"
- board text added: "Castellated pads:"
- board text added: "Copper Finish:"
- board text added: "Copper Layer Count:"
- board text added: "Edge card connectors:"
- board text added: "Impedance Control:"
- board text added: "Min hole diameter:"
- board text added: "Min track/spacing:"
- board text added: "No"
- board text added: "None"
- board text added: "Plated Board Edge:"
- board text added: "rev. 1.2 2024"
- board text removed: "rev. 1.1 2024"
